File: Car Schematic/12VElectronics.kicad_sch (KiCad schematic)
At the start: 2 parts

Commit message: wip commit car schematic
Parts:
- removed BT?: 12V AUX Battery, symbol Device:Battery
- added D?: DIODE, symbol pspice:DIODE
- added D?: FUN LIGHTS!, symbol Device:LED
- added F? (x12): Fuse, symbol Device:Fuse
- added F?: 3A, symbol Device:Fuse
- added JP?: Jumper_2_Bridged, symbol Jumper:Jumper_2_Bridged
- added K? (x2): 12V, 50A, symbol Relay:G5Q-1A
- added LA?: INTERIOR LIGHTS, symbol Device:Lamp
- added LA?: FRONT LEFT TURN LIGHT, symbol Device:Lamp
- added LA?: FRONT RIGHT TURN LIGHT, symbol Device:Lamp
- added LA?: RUNNING LIGHTS, symbol Device:Lamp
- added LA?: LEFT HEAD LIGHT, symbol Device:Lamp
- added LA?: RIGHT HEAD LIGHT, symbol Device:Lamp
- added LS?: HORN, symbol Device:Speaker
- added LS?: PASSENGER BELL, symbol Device:Speaker
- added M?: HEATER BLOWER, symbol Motor:Fan_IEC60617
- added M?: WINDSHIELD WIPER MOTOR, symbol Motor:Motor_DC_ALT
- added R?: RADIO, symbol Device:R
- added R?: PASSENGER SEAT HEATER, symbol Device:Heater
- added R?: CB RADIO, symbol Device:R
- added R?: DRIVER SEAT HEATER, symbol Device:Heater
- added R?: USB-C CHARGER, symbol Device:R
- added SW?: HEAD LIGHT SWITCH, symbol Switch:SW_SPST
- added SW?: WINDSHIELD WIPER SWITCH, symbol Switch:SW_DP3T
- added SW?: HEATER SWITCH, symbol Switch:SW_SPST
- added SW?: PASSENGER BELL SWITCH, symbol Switch:SW_MEC_5G
- added SW?: USB-C SWITCH, symbol Switch:SW_SPST
- added SW?: INTERIOR LIGHT SWITCH, symbol Switch:SW_SPST
- added SW?: AUX LIGHTS SWITCH, symbol Switch:SW_SPST
- added SW?: TURN SIGNAL, symbol Switch:SW_SPDT_MSM
- added SW?: BRAKE PEDAL, symbol Switch:SW_MEC_5G
- added SW?: DRIVER SEAT HEATER, symbol Switch:SW_SPST
- added SW?: HORN SWITCH, symbol Switch:SW_MEC_5G
- added SW?: RADIO SWITCH, symbol Switch:SW_SPST
- added SW?: PASSENGER SEAT HEATER, symbol Switch:SW_SPST
Connections:
- net +12V: now also F?.1, K?.3, K?.3
- net GNDPWR: now also D?.1 (K), K?.1, K?.1, LA?.1 (-), LA?.1 (-), LA?.1 (-), LA?.1 (-), LA?.1 (-), LA?.1 (-), LS?.2, LS?.2, M?.2 (-), M?.2 (-), R?.2, R?.2, R?.2, R?.2, R?.2
- net KEY_OFF: now reaches SW?.1 (OFF)
- net KEY_AUX: now reaches SW?.2 (AUX)
- net IGNITION_KEY_INPUT: now reaches SW?.3
- net IGNITION_KEY_INPUT: now also F?.2
- net KEY_ON: now reaches SW?.4 (ON)
- net KEY_ON: now also D?.1 (K), K?.5
- new net: LA?.2 (+), SW?.2 (B)
- new net: M?.1 (+), SW?.1 (OFF), SW?.2 (INT), SW?.4 (ON)
- new net: F?.2, SW?.3
- new net: M?.1 (+), SW?.2 (B)
- new net: F?.2, SW?.1 (A), SW?.1 (A), SW?.1 (A), SW?.2 (A), SW?.2 (A), SW?.2 (A)
- new net: LS?.1, SW?.3 (B), SW?.4 (B) (x2)
- new net: R?.1, R?.1, SW?.2 (B)
- new net: R?.1, SW?.2 (B) (x3)
- new net: D?.2 (A), SW?.2 (B)
- new net: SW?.3 (B), SW?.4 (B)
- new net +12C: F?.1
- new net AUX LIGHTS: F?.2, SW?.1 (A)
- new net AUX_POWER_RELAYED: F?.1, F?.1, F?.1, K?.2
- new net GAUGE_CLUSTER_POWER: F?.2
- new net HEAD_LIGHT_POWER_SWITCHED: JP?.2 (B), LA?.2 (+), LA?.2 (+), LA?.2 (+), SW?.2 (B)
- new net INTERIOR_LIGHTS_AND_HEATER: F?.2, SW?.1 (A), SW?.1 (A)
- new net KEY AUX: D?.2 (A), K?.5
- new net LEFT_TURN_SIGNAL: LA?.2 (+), SW?.1
- new net LIGHTS AND SIGNALS: F?.2, SW?.1 (A), SW?.2
- new net ON_POWER_RELAYED: F?.1, F?.1, F?.1, F?.1, F?.1, F?.1, F?.1, F?.1, K?.2
- new net RADIO: F?.2, SW?.1 (A)
- new net RIGHT_TURN_SIGNAL: LA?.2 (+), SW?.3
- new net RUNNING_LIGHT_POWER: JP?.1 (A)
- new net SEAT HEATERS: F?.2, SW?.1 (A), SW?.1 (A)
- new net USB_C_POWER: F?.2, SW?.1 (A)
Other:
- note added: "100W"
- note added: "10W"
- note added: "15W"
- note added: "250W"
- note added: "25W"
- note added: "30W"
- note added: "50W"
- note added: "55W"
- note added: "70W"
- note added: "75W"
- note added: "ADD IN OTHER PINS THAT ARE ON HEATER BLOWER"
- note added: "FRONT ELECTRIC PANEL 1"
- note removed: "(CONNECTED TO CHASSIS)"
- note removed: "(TO DC/DC CHARGER)"
- moved on the sheet: SW?A

Commit message: lots of changes
Other:
- added sheet Front Electrical Panel 2\Gauge Cluster (Gauge Panel.kicad_sch)
- company: (none) -> MATTHEW BRYANT-HEIDEBRECHT
- title: (none) -> ELECTRAVAN 500 SCHEMATIC

Commit message: updating more things!
Parts:
- removed F? (x3): Fuse, symbol Device:Fuse
- removed JP?: Jumper_2_Bridged, symbol Jumper:Jumper_2_Bridged
- added D?: LIGHT BAR, symbol Device:LED
- added F? (x4): Fuse, symbol Device:Fuse
- added J?: 12V OUTLET, symbol Connector:Conn_Coaxial_Power
- added JP? (x2): Jumper_2_Bridged, symbol Jumper:Jumper_2_Bridged
- added R?: CELL BOOSTER, symbol Device:R
- added R?: PHONE CHARGER, symbol Device:R
- added R?: WIFI HOTSPOT, symbol Device:R
- added SW?: CELL BOOSTER SWITCH, symbol Switch:SW_SPST
- added SW?: 12V OUTLET SWITCH, symbol Switch:SW_SPST
- added SW?: PHONE CHARGER SWITCH, symbol Switch:SW_SPST
- added SW?: LIGHT BAR SWITCH, symbol Switch:SW_SPST
Connections:
- net BRAKE_LIGHT_POWER: now also JP?.1 (A)
- net BRAKE_PEDAL_SIGNAL: now also JP?.2 (B)
- net GNDPWR: now also D?.1 (K), J?.2 (Ext), R?.2, R?.2, R?.2
- net HEAD_LIGHT_POWER_SWITCHED: now also JP?.2 (B)
- net ON_POWER_RELAYED: now also F?.1, F?.1, F?.1
- net RUNNING_LIGHT_POWER: now also JP?.1 (A)
- new net: R?.1, R?.1, SW?.2 (B)
- new net: J?.1 (In), SW?.2 (B)
- new net: F?.2, SW?.1 (A) (x3)
- new net: R?.1, SW?.2 (B)
- new net: D?.2 (A), SW?.2 (B)
- new net 12V OUTLET: F?.2, SW?.1 (A)
Other:
- note added: "(to B1)"
- note added: "(to C6)"
- note added: "So all Aux circuits stay active while car is on"
- note added: "The below end up going to the engine compartment"
- moved on the sheet: D?, F?, LA?, R?, SW?
