File: Car Schematic/Car Schematic.kicad_sch (KiCad schematic)
At the start: 20 parts

Commit message: updates
Parts:
- added F?: 12V, 80A, symbol Device:Fuse
- added K?: DISCHARGE ENABLE RELAY, symbol Relay:G5Q-1A
- gave numbers to parts that had none: 3
Connections:
- net GNDS is gone; now on net MTR_THERM_SIGNAL: M?.~ (THERMISTOR_SIG)
- net MTR_THERM_SIG is gone; now on net MTR_THERM_SIGNAL: M?.~ (THERMISTOR_SIG)
- net +12V: now also F?.2; no longer IC?.~ (PE_(GND))
- net 0_GA: no longer BT?.~ (THERM2-)
- net CURRENT_CHANNEL_GND: no longer U?.~ (THERM_8_RTN)
- net CURRENT_CHANNEL_HIGH: no longer U?.~ (THERM_8_RTN)
- net CURRENT_CHANNEL_LOW: no longer U?.~ (THERM_8_RTN)
- net CURRENT_SENSE_+VDC: no longer U?.~ (THERM_8_RTN)
- net GNDPWR: now also M?.~ (THERMISTOR_SIG)
- net at W?.~ (BUS_2): now also BT?.~ (THERM2-); no longer BT?.~ (THERM2-) (x4)
- net MTR_THERM_SIGNAL: now reaches M?.~ (THERMISTOR_SIG)
- net MTR_THERM_SIGNAL: no longer IC?.~ (VDC-)
- new net: BT?.~ (THERM2-), W?.~ (BUS_2) (x4)
- new net: BT?.~ (THERM2-), IC?.~ (SENSE_SIGNAL_LOW)
- new net: IC?.~ (VDC-), K?.3
- new net: IC?.~ (VDC-), M?.~ (THERMISTOR_SIG) (x2)
- new net: F?.1, IC?.~ (PE_(GND))
- new net CELL_19-: BT?.~ (THERM2-)
- no-connect marks 0 -> 10
Other:
- added sheet 12V Electronics (12VElectronics.kicad_sch)
- note added: "(CONNECTED TO CHASSIS)"
- note added: "(TO 12V SCHEMATIC)"
- note added: "BATTERY PACK"
- note added: "Wires and Buses represent the physical wire configuration. Buses represent wire looms Thick wires ( ) represent low gauge (big) wires and small wires ( ) represent small wires (Parenthesis indicate soft references and may not be correct through updates)"
- moved on the sheet: F?, K?, M?, RV?, SW?, U?

Commit message: wip commit car schematic
Parts:
- removed C?: J1772_charge_connector, symbol matt's custom carp:J1772_charge_connector
- removed M?: BALDOR_DC_MOTOR, symbol matt's custom carp:BALDOR_DC_MOTOR
- added BT?: 12V AUX Battery, symbol Device:Battery
- added F?: 12V, 5A, symbol Device:Fuse
- added JP?: Jumper_2_Bridged, symbol Jumper:Jumper_2_Bridged
- added K?: RELAY, 12V, symbol Relay:G5Q-1A
- added SW?: INERTIA SWITCH, symbol Switch:SW_Push_Open
- added TH1, TH2, TH3, TH4, TH5, TH6, TH7, TH8: Thermistor, symbol Device:Thermistor
- added U?: LOW VOLTAGE CUTOFF, symbol Analog_Switch:ADG417BN
Connections:
- net ALWAYS_ON_POWER is gone; now on net THERM_8_RTN: U?.~ (THERM_8_RTN)
- net J1772_CP is gone; now on net THERM_8_RTN: U?.~ (THERM_8_RTN)
- net J1772_PD is gone; now on net THERM_8_RTN: U?.~ (THERM_8_RTN)
- net +12V: now also BT?.1 (+), K?.2, U?.1, U?.6
- net CHARGE_POWER: now also F?.1; no longer IC?.~ (PE_(GND))
- net DISCHARGE_ENABLE: now also K?.1
- net GNDPWR: now also K?.1, BT?.2 (-)
- net READY_POWER: now also JP?.2 (B)
- net THERM_1+: now also TH1.1
- net THERM_1_RTN: now also TH1.2
- net THERM_2+: now also TH2.1
- net THERM_2_RTN: now also TH2.2
- net THERM_3+: now also TH3.1
- net THERM_3_RTN: now also TH3.2
- net THERM_4+: now also TH4.1
- net THERM_4_RTN: now also TH4.2
- net THERM_5+: now also TH5.1
- net THERM_5_RTN: now also TH5.2
- net THERM_6+: now also TH6.1
- net THERM_6_RTN: now also TH6.2
- net THERM_7+: now also TH7.1
- net THERM_7_RTN: now also TH7.2
- net THERM_8+: now also TH8.1
- net THERM_8_RTN: now also TH8.2
- net at W?.~ (BUS_2): now also BT?.~ (THERM2-); no longer BT?.~ (THERM2-) (x4)
- net M2: now reaches IC?.~ (VDC-)
- net at K?.3: now also SW?.1 (A); no longer IC?.~ (VDC-)
- net +12C: now reaches K?.2
- net +12C: now also U?.~ (THERM_8_RTN), U?.8
- net KEY_ON: now reaches K?.5
- net KEY_ON: now also JP?.1 (A)
- net CHARGE RELAY OUT: now reaches K?.5
- net CHARGE RELAY OUT: now also IC?.~ (VDC-), SW?.2 (B)
- new net: BT?.~ (THERM2-), W?.~ (BUS_2) (x4)
- new net: BT?.~ (THERM2-), IC?.~ (SENSE_SIGNAL_LOW)
- new net: F?.2, IC?.~ (PE_(GND))
- new net AC_LINE: IC?.~ (PE_(GND))
- new net AC_NEUTRAL: IC?.~ (PE_(GND))
- new net AC_PE: IC?.~ (PE_(GND))
- new net CONTROL PILOT: U?.~ (THERM_8_RTN)
- new net M1: IC?.~ (VDC-)
- new net PROXIMITY DETECT: U?.~ (THERM_8_RTN)
Other:
- sheet 12V Electronics renamed Front Electronic Panel
- added sheet Engine Compartment (Engine Compartment.kicad_sch)
- added sheet Front Electrical Panel 2\Gauge Cluster (Gauge Panel.kicad_sch)
- added sheet Upper Indicator Panel (uppder_indicator_panel.kicad_sch)
- note added: "BATTERY BOX SCHEMATIC"
- note added: "TO ENGINE COMPARTMENT"
- note added: "TO FRONT PANEL"
- note added: "TODO"
- note removed: "(TO 12V SCHEMATIC)"
- moved on the sheet: F?, IC?, K?

Commit message: lots of changes
Parts:
- removed BT? (x6): TESLA_24_V_MODULE, symbol matt's custom carp:TESLA_24_V_MODULE
- removed BT?: 12V AUX Battery, symbol Device:Battery
- removed F?: Fuse, 400VDC, 1000A, symbol Device:Fuse
- removed F?: 12V, 80A, symbol Device:Fuse
- removed F?: 12V, 5A, symbol Device:Fuse
- removed IC?: CURRENT_SENSOR, symbol matt's custom carp:CURRENT_SENSOR
- removed IC?: ZEVA_MC1000C, symbol matt's custom carp:ZEVA_MC1000C
- removed IC?: SEV33ADE-144V, symbol matt's custom carp:SEV33ADE-144V
- removed JP?: Jumper_2_Bridged, symbol Jumper:Jumper_2_Bridged
- removed K?: DISCHARGE ENABLE RELAY, symbol Relay:G5Q-1A
- removed K?: RELAY, 12V, symbol Relay:G5Q-1A
- removed K?: CONTACTOR, 400V, 1000A, symbol Relay:G5Q-1A
- removed RV?: THROTTLE, symbol Device:R_Potentiometer_US
- removed SW?: INERTIA SWITCH, symbol Switch:SW_Push_Open
- removed SW?: MAINTENANCE_SW_LOCKOUT, symbol Switch:SW_SPST
- removed TH1, TH2, TH3, TH4, TH5, TH6, TH7, TH8: Thermistor, symbol Device:Thermistor
- removed U?: LOW VOLTAGE CUTOFF, symbol Analog_Switch:ADG417BN
- removed U?: ORION_36S_BMS, symbol matt's custom carp:ORION_36S_BMS
- removed W? (x4): TESLA_MODULE_BUSBAR, symbol matt's custom carp:TESLA_MODULE_BUSBAR
Connections:
- no-connect marks 10 -> 0
Other:
- removed sheet Front Electrical Panel 2\Gauge Cluster
- added sheet Battery Box (battery_box.kicad_sch)
- note added: "BATTERY BOX TO FRONT PANEL HARNESS"
- note added: "ENGINE COMPARTMENT TO BATTERY BOX HARNESS"
- note added: "GAUGE PANEL GAUGE ARBITRATOR 12V FUSES CONTROL SWITCHES HEATER USB CHARGER PHONE CHARGER"
- note added: "HVDC BATTERY BMS CHARGER DC/DC CONVERTER AUX BATTERY (12V) MOTOR CONTROLLER"
- note added: "MOTOR TRANSMISSION REAR LIGHTS J1772 CHARGE PLUG"
- note added: "SCHEMATIC LOATION DEFINITION HARNESS OVERVIEW SCHEMATIC INTERCONNECT DEFINITION"
- note added: "WARNING INDICATORS SWITCHES CLOCK"
- note removed: "(CONNECTED TO CHASSIS)"
- note removed: "BATTERY BOX SCHEMATIC"
- note removed: "BATTERY PACK"
- note removed: "TO ENGINE COMPARTMENT"
- note removed: "TO FRONT PANEL"
- note removed: "TODO"
- note removed: "Wires and Buses represent the physical wire configuration. Buses represent wire looms Thick wires ( ) represent low gauge (big) wires and small wires ( ) represent small wires (Parenthesis indicate soft references and may not be correct through updates)"
- company: (none) -> MATTHEW BRYANT-HEIDEBRECHT
- title: (none) -> ELECTRAVAN 500 SCHEMATIC

Commit message: updating more things!
Other:
- note added: "GAUGE PANEL GAUGE ARBITRATOR 12V FUSES CONTROL SWITCHES HEATER USB CHARGER PHONE CHARGER FRONT LIGHTS"
- note removed: "GAUGE PANEL GAUGE ARBITRATOR 12V FUSES CONTROL SWITCHES HEATER USB CHARGER PHONE CHARGER"
