File: Car Schematic/Gauge Panel.kicad_sch (KiCad schematic)
At the start: 19 parts

Commit message: lots of changes
Other:
- note added: "Wires and Buses represent the physical wire configuration. Buses represent wire looms Thick wires ( ) represent low gauge (big) wires and small wires ( ) represent small wires (Parenthesis indicate soft references and may not be correct through updates)"
- company: (none) -> MATTHEW BRYANT-HEIDEBRECHT
- title: (none) -> ELECTRAVAN 500 SCHEMATIC
Changed lines of the file:
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@@
 (kicad_sch (version 20211123) (generator eeschema)
-  (paper "B")
+  (paper "A")
+  (title_block
+    (title "ELECTRAVAN 500 SCHEMATIC")
+    (date "2022-11-23")
+    (rev "0.1")
+    (company "MATTHEW BRYANT-HEIDEBRECHT")
+    (comment 1 "(PARENTHESIS REPRESENTS SOFT REFERENCES AND MAY NOT BE CORRECT THROUGH UPDATES)")
+    (comment 2 "THICK WIRES REPRESENT LOW GAUGE WIRES, SMALL WIRES REPRESENT HIGH GAUGE WIRES")
+    (comment 3 "BUSES REPRESENT WIRE LOOMS ")
+    (comment 4 "WIRES AND BUSES REPRESENT THE PHYSICAL WIRE CONFIGURATIONS")
+  )
   (junction (at 127 207.645) (diameter 0) (color 0 0 0 0)
   )
@@
     (stroke (width 0) (type default) (color 0 0 0 0))
   )
+  (wire (pts (xy 27.305 25.4) (xy 38.735 25.4))
+    (stroke (width 0.5) (type default) (color 0 0 0 0))
+  )
   (wire (pts (xy 207.645 100.33) (xy 207.645 116.205))
     (stroke (width 0) (type default) (color 0 0 0 0))
@@
   )
   (wire (pts (xy 127 217.17) (xy 127 215.265))
+    (stroke (width 0) (type default) (color 0 0 0 0))
+  )
+  (wire (pts (xy 90.17 25.4) (xy 109.22 25.4))
     (stroke (width 0) (type default) (color 0 0 0 0))
   )
@@
     (effects (font (size 5.08 5.08)) (justify right bottom))
   )
+  (text "Wires and Buses represent the physical wire configuration.\nBuses represent wire looms\nThick wires (		) represent low gauge (big) wires and small wires (		) represent small wires\n(Parenthesis indicate soft references and may not be correct through updates)"
+    (at 13.97 27.94 0)
+    (effects (font (size 1.27 1.27)) (justify left bottom))
+  )
   (label "BATTERY_TEMP_SELECT_SIGNAL" (at 87.63 204.47 180)

Commit message: updating more things!
Parts:
- removed R? (x6): R, symbol Device:R
- added SW?: MAX MOTOR CURRENT SWITCH, symbol Switch:SW_Rotary12
- added SW?: CONSUMPTION GAUGE DISPLAY SWITCH, symbol Switch:SW_Rotary12
- added SW?: OTHER TEMP DISPLAY SELECT SWITCH, symbol Switch:SW_Rotary12
- added U?: OTHER TEMP GAUGE, symbol matt's custom carp:GAUGE
- added U?: MOTOR AMP GAUGE, symbol matt's custom carp:GAUGE
- added U?: HV BATT SOC GAUGE, symbol matt's custom carp:GAUGE
- SW?: value BATTERY TEMP SELECT SWITCH -> BATTERY TEMP DISPLAY SELECT SWITCH
- U?: value CLOCK -> 12V VOLT GAUGE
Connections:
- net AUX_POWER_RELAYED: no longer SW?.1
- net GND: no longer SW?.12
- net GNDPWR: now also U?. (SIGNAL)
- net BATTERY_TEMP_SELECT_SIGNAL: no longer names the net of SW?.13
- new net ALL TIME: SW?.4
- new net BATT CYCLE: SW?.3
- new net BENNI: SW?.4
- new net BMS AUX 1: SW?.5
- new net BMS AUX 2... AND SO ON: SW?.6
- new net BMS TEMP: SW?.2
- new net CHARGER TEMP: SW?.4
- new net CTLR TEMP: SW?.3
- new net MEDIUM: SW?.3
- new net RABBIT: SW?.5
- new net TRIP: SW?.2
- new net TURTLE: SW?.2
- new net WARP SPEED: SW?.6
Other:
- note added: "SELECT THERMISTOR TO DISPLAY, 2 EXTRA OPTIONS FOR: MAX TEMP MIN TEMP"
- note removed: "Wires and Buses represent the physical wire configuration. Buses represent wire looms Thick wires ( ) represent low gauge (big) wires and small wires ( ) represent small wires (Parenthesis indicate soft references and may not be correct through updates)"
- moved on the sheet: LA?, R?, RV?, SW?, U?
