File: Car Schematic/battery_box.kicad_sch (KiCad schematic)
At the start: 34 parts

Commit message: updating more things!
Parts:
- removed F?: Fuse, 400VDC, 1000A, symbol Device:Fuse
- removed JP?: Jumper_2_Bridged, symbol Jumper:Jumper_2_Bridged
- removed SW?: MAINTENANCE_SW_LOCKOUT, symbol Switch:SW_SPST
- added D?: BATTERY BOX LIGHTS, symbol Device:LED
- added F?: 200V, 30A, symbol Device:Fuse
- added F?: Fuse, 400VDC, 1000A, symbol Device:Fuse
- added F? (x2): Fuse, symbol Device:Fuse
- added F?: 12V, 10A, symbol Device:Fuse
- added F?: 12V, 100A, symbol Device:Fuse
- added J?: 12V OUTLET, symbol Connector:Conn_Coaxial_Power
- added J?: CAN_DB9_Female, symbol Connector:DB9_Female
- added JP? (x3): Jumper_2_Bridged, symbol Jumper:Jumper_2_Bridged
- added R?: PRECHARGER RESISTOR, symbol Device:R
- added R?: 12V AMP SENSE SHUNT, symbol Device:R_Shunt
- added SW?: MAINTENANCE_SW_LOCKOUT, symbol Switch:SW_SPST
- added SW?: BATTERY BOX LIGHT SWITCH, symbol Switch:SW_SPST
- added SW?: 12V OUTLET SWITCH, symbol Switch:SW_SPST
- BT?: value 12V AUX Battery -> AUX Battery
- K?: value RELAY, 12V -> PRECHARGER RELAY, 12V IN, 400VDC OUT
Connections:
- net DC/DC_ACTIVATE is gone; now on net GNDPWR: IC?.~ (PE_(GND))
- net +12C: now also JP?.2 (B); no longer U?.~ (THERM_8_RTN)
- net +12V: now also F?.1, F?.1, F?.1, F?.1; no longer BT?.1 (+), U?.1, U?.6
- net +VSW: now also K?.1, F?.2; no longer IC?.~ (PE_(GND))
- net 0_GA: now also F?.1; no longer IC?.~ (SENSE_SIGNAL_LOW)
- net CAN1_H: now also J?.2
- net CAN1_L: now also J?.3
- net DC/DC ACTIVATE: now also IC?.~ (PE_(GND)), JP?.1 (A)
- net GNDPWR: now also D?.1 (K), J?.2 (Ext), R?.1; no longer BT?.2 (-)
- net KEY_ON: now also JP?.2 (B), JP?.2 (B)
- net READY_POWER: now also JP?.1 (A)
- net at W?.~ (BUS_2): now also BT?.~ (THERM2-); no longer BT?.~ (THERM2-) (x4)
- net at K?.5: now also R?.2
- net at K?.3: now also BT?.~ (THERM2-), R?.1
- new net: IC?.~ (SENSE_SIGNAL_LOW), SW?.1 (A)
- new net: BT?.~ (THERM2-), SW?.2 (B)
- new net: BT?.~ (THERM2-), W?.~ (BUS_2) (x4)
- new net: F?.1, IC?.~ (PE_(GND))
- new net: J?.1 (In), SW?.2 (B)
- new net: F?.2, IC?.~ (SENSE_SIGNAL_LOW)
- new net: F?.2, SW?.2 (B)
- new net: D?.2 (A), SW?.1 (A)
- new net: F?.2, U?.1, U?.6
- new net: F?.2, SW?.1 (A)
- new net: BT?.2 (-), R?.4
- new net: BT?.1 (+), F?.2
- new net ALWAYS_ON_POWER: JP?.1 (A), U?.~ (THERM_8_RTN)
- new net CAN1_GND: J?.9
Other:
- note added: "(look down and left)"
- note added: "(look up and right)"
- note added: "(to A3 too)"
- note added: "(to G3)"
- note added: "12V "ALWAYS ON" POWER OUTPUT"
- note added: "12V POWER OUTPUT"
- note added: "LEAD ACID 12V, 40AH"
- note added: "NEED PRECHARGER CONTROL"
- note removed: "TO FRONT PANEL"
- note removed: "TODO"
- moved on the sheet: K?, U?A
