File: Car Schematic/uppder_indicator_panel.kicad_sch (KiCad schematic)
At the start: 9 parts

Commit message: lots of changes
Other:
- note added: "Wires and Buses represent the physical wire configuration. Buses represent wire looms Thick wires ( ) represent low gauge (big) wires and small wires ( ) represent small wires (Parenthesis indicate soft references and may not be correct through updates)"
- company: (none) -> MATTHEW BRYANT-HEIDEBRECHT
- title: (none) -> ELECTRAVAN 500 SCHEMATIC
Changed lines of the file:
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@@
 (kicad_sch (version 20211123) (generator eeschema)
-  (paper "B")
-  (bus_entry (at 17.78 38.735) (size 2.54 2.54)
+  (paper "A")
+  (title_block
+    (title "ELECTRAVAN 500 SCHEMATIC")
+    (date "2022-11-23")
+    (rev "0.1")
+    (company "MATTHEW BRYANT-HEIDEBRECHT")
+    (comment 1 "(PARENTHESIS REPRESENTS SOFT REFERENCES AND MAY NOT BE CORRECT THROUGH UPDATES)")
+    (comment 2 "THICK WIRES REPRESENT LOW GAUGE WIRES, SMALL WIRES REPRESENT HIGH GAUGE WIRES")
+    (comment 3 "BUSES REPRESENT WIRE LOOMS ")
+    (comment 4 "WIRES AND BUSES REPRESENT THE PHYSICAL WIRE CONFIGURATIONS")
+  )
+  (bus_entry (at 15.24 51.435) (size 2.54 2.54)
     (stroke (width 0) (type default) (color 0 0 0 0))
   )
-  (bus_entry (at 17.78 45.085) (size 2.54 2.54)
+  (bus_entry (at 15.24 57.785) (size 2.54 2.54)
     (stroke (width 0) (type default) (color 0 0 0 0))
   )
-  (bus_entry (at 17.78 41.91) (size 2.54 2.54)
+  (bus_entry (at 15.24 54.61) (size 2.54 2.54)
     (stroke (width 0) (type default) (color 0 0 0 0))
   )
-  (bus_entry (at 17.78 32.385) (size 2.54 2.54)
+  (bus_entry (at 15.24 45.085) (size 2.54 2.54)
     (stroke (width 0) (type default) (color 0 0 0 0))
   )
-  (bus_entry (at 17.78 35.56) (size 2.54 2.54)
+  (bus_entry (at 15.24 48.26) (size 2.54 2.54)
     (stroke (width 0) (type default) (color 0 0 0 0))
   )
-  (bus (pts (xy 22.225 20.32) (xy 17.78 20.32))
+  (bus (pts (xy 19.685 33.02) (xy 15.24 33.02))
     (stroke (width 0) (type default) (color 0 0 0 0))
   )
-  (bus (pts (xy 17.78 35.56) (xy 17.78 38.735))
+  (bus (pts (xy 15.24 48.26) (xy 15.24 51.435))
     (stroke (width 0) (type default) (color 0 0 0 0))
   )
-  (bus (pts (xy 17.78 32.385) (xy 17.78 35.56))
+  (bus (pts (xy 15.24 45.085) (xy 15.24 48.26))
     (stroke (width 0) (type default) (color 0 0 0 0))
   )
@@
     (stroke (width 0) (type default) (color 0 0 0 0))
   )
-  (wire (pts (xy 20.32 38.1) (xy 43.815 38.1))
+  (wire (pts (xy 17.78 50.8) (xy 41.275 50.8))
     (stroke (width 0) (type default) (color 0 0 0 0))
   )
-  (bus (pts (xy 17.78 41.91) (xy 17.78 45.085))
+  (bus (pts (xy 15.24 54.61) (xy 15.24 57.785))
     (stroke (width 0) (type default) (color 0 0 0 0))
   )
-  (wire (pts (xy 20.32 34.925) (xy 43.815 34.925))
+  (wire (pts (xy 17.78 47.625) (xy 41.275 47.625))
     (stroke (width 0) (type default) (color 0 0 0 0))
   )
-  (wire (pts (xy 20.32 41.275) (xy 43.815 41.275))
+  (wire (pts (xy 17.78 53.975) (xy 41.275 53.975))
     (stroke (width 0) (type default) (color 0 0 0 0))
   )
-  (bus (pts (xy 17.78 38.735) (xy 17.78 41.91))
+  (bus (pts (xy 15.24 51.435) (xy 15.24 54.61))
     (stroke (width 0) (type default) (color 0 0 0 0))
   )
-  (bus (pts (xy 17.78 20.32) (xy 17.78 32.385))
+  (bus (pts (xy 15.24 33.02) (xy 15.24 45.085))
     (stroke (width 0) (type default) (color 0 0 0 0))
   )
-  (wire (pts (xy 20.32 47.625) (xy 43.815 47.625))
+  (wire (pts (xy 17.78 60.325) (xy 41.275 60.325))
     (stroke (width 0) (type default) (color 0 0 0 0))
   )
-  (wire (pts (xy 20.32 44.45) (xy 43.815 44.45))
+  (wire (pts (xy 26.035 17.78) (xy 37.465 17.78))
+    (stroke (width 0.5) (type default) (color 0 0 0 0))
+  )
+  (wire (pts (xy 17.78 57.15) (xy 41.275 57.15))
     (stroke (width 0) (type default) (color 0 0 0 0))
   )
-  (label "HEAD_LIGHT_POWER_SWITCHED" (at 21.59 41.275 0)
+  (wire (pts (xy 88.9 17.78) (xy 107.95 17.78))
+    (stroke (width 0) (type default) (color 0 0 0 0))
+  )
+  (text "Wires and Buses represent the physical wire configuration.\nBuses represent wire looms\nThick wires (		) represent low gauge (big) wires and small wires (		) represent small wires\n(Parenthesis indicate soft references and may not be correct through updates)"
+    (at 12.7 20.32 0)
     (effects (font (size 1.27 1.27)) (justify left bottom))
   )
-  (label "CAN1_L" (at 21.59 47.625 0)
+  (label "HEAD_LIGHT_POWER_SWITCHED" (at 19.05 53.975 0)
     (effects (font (size 1.27 1.27)) (justify left bottom))
   )
-  (label "GAUGE_CLUSTER_POWER" (at 21.59 38.1 0)
+  (label "CAN1_L" (at 19.05 60.325 0)
     (effects (font (size 1.27 1.27)) (justify left bottom))
   )
-  (label "CAN1_H" (at 21.59 44.45 0)
+  (label "GAUGE_CLUSTER_POWER" (at 19.05 50.8 0)
+    (effects (font (size 1.27 1.27)) (justify left bottom))
+  )
+  (label "CAN1_H" (at 19.05 57.15 0)
     (effects (font (size 1.27 1.27)) (justify left bottom))
   )
@@
     (effects (font (size 1.27 1.27)) (justify left bottom))
   )
-  (label "BMS_RESET_SIG" (at 21.59 34.925 0)
+  (label "BMS_RESET_SIG" (at 19.05 47.625 0)
     (effects (font (size 1.27 1.27)) (justify left bottom))
   )
-  (global_label "FRONT_TO_UPPER_PANEL_BUS" (shape passive) (at 22.225 20.32 0) (fields_autoplaced)
+  (global_label "FRONT_TO_UPPER_PANEL_BUS" (shape passive) (at 19.685 33.02 0) (fields_autoplaced)
     (effects (font (size 1.27 1.27)) (justify left))
-    (property "Intersheet References" "${INTERSHEET_REFS}" (id 0) (at 52.6706 20.2406 0)
+    (property "Intersheet References" "${INTERSHEET_REFS}" (id 0) (at 50.1306 32.9406 0)
       (effects (font (size 1.27 1.27)) (justify left) hide)
     )
